Commit message: Add reusable rocker macro with left and right instances

File: src/my_rover_description/urdf/rocker.xacro (robot description, xacro)
@@ -6,6 +6,7 @@
         <origin xyz="0 0 0" rpy="0 0 0"/>
         <geometry>
-          <box size="0.30 0.05 0.05"/>
-        </geometry>
+  <mesh filename="package://my_rover_description/meshes/visual/rocker_link.stl"
+        scale="0.001 0.001 0.001"/>
+</geometry>
         <material name="blue">
           <color rgba="0.1 0.3 1.0 1.0"/>
