Commit message: Add base_link mesh and verify RViz visualization

File: src/my_rover_description/urdf/my_rover.urdf.xacro (robot description, xacro)
@@ -6,6 +6,7 @@
       <origin xyz="0 0 0" rpy="0 0 0"/>
       <geometry>
-        <box size="0.6 0.4 0.1"/>
-      </geometry>
+    <mesh filename="package://my_rover_description/meshes/visual/base_link.stl"
+          scale="0.001 0.001 0.001"/>
+</geometry>
       <material name="gray">
         <color rgba="0.7 0.7 0.7 1.0"/>

Commit message: Move robot dimensions into properties.xacro

File: src/my_rover_description/urdf/my_rover.urdf.xacro (robot description, xacro)
@@ -4,4 +4,5 @@
     <xacro:include filename="rocker.xacro"/>
     <xacro:include filename="bogie.xacro"/>
+    <xacro:include filename="properties.xacro"/>
   <link name="base_link">
     <visual>
@@ -17,18 +18,18 @@
   </link>
   <xacro:rocker
-      name="left_rocker"
-      parent="base_link"
-      xyz="0 0.25 0"/>
-  <xacro:rocker
-      name="right_rocker"
-      parent="base_link"
-      xyz="0 -0.25 0"/>
+    name="left_rocker"
+    parent="base_link"
+    xyz="${rocker_x} ${rocker_y} ${rocker_z}"/>
+<xacro:rocker
+    name="right_rocker"
+    parent="base_link"
+    xyz="${rocker_x} ${-rocker_y} ${rocker_z}"/>
   <xacro:bogie
-      name="left_bogie"
-      parent="left_rocker"
-      xyz="0.25 0 -0.05"/>
-  <xacro:bogie
-      name="right_bogie"
-      parent="right_rocker"
-      xyz="0.25 0 -0.05"/>
+    name="left_bogie"
+    parent="left_rocker"
+    xyz="${bogie_x} ${bogie_y} ${bogie_z}"/>
+<xacro:bogie
+    name="right_bogie"
+    parent="right_rocker"
+    xyz="${bogie_x} ${bogie_y} ${bogie_z}"/>
 </robot>

File: src/my_rover_description/urdf/properties.xacro (robot description, xacro)
@@ -1,5 +1,13 @@
 <?xml version="1.0"?>
 <robot xmlns:xacro="http://www.ros.org/wiki/xacro">
-    <xacro:property name="mesh_path"
-                    value="package://my_rover_description/meshes/visual"/>
+  <!-- Mesh Scale -->
+  <xacro:property name="mesh_scale" value="0.001 0.001 0.001"/>
+  <!-- Rocker Position -->
+  <xacro:property name="rocker_x" value="0.0"/>
+  <xacro:property name="rocker_y" value="0.25"/>
+  <xacro:property name="rocker_z" value="0.0"/>
+  <!-- Bogie Position -->
+  <xacro:property name="bogie_x" value="0.25"/>
+  <xacro:property name="bogie_y" value="0.0"/>
+  <xacro:property name="bogie_z" value="-0.05"/>
 </robot>

Commit message: Add rover URDF and Gazebo simulation

File: src/my_rover_description/urdf/my_rover.urdf.xacro (robot description, xacro)
@@ -2,34 +2,85 @@
 <robot name="my_rover"
        xmlns:xacro="http://www.ros.org/wiki/xacro">
-    <xacro:include filename="rocker.xacro"/>
-    <xacro:include filename="bogie.xacro"/>
-    <xacro:include filename="properties.xacro"/>
-  <link name="base_link">
-    <visual>
-      <origin xyz="0 0 0" rpy="0 0 0"/>
-      <geometry>
-    <mesh filename="package://my_rover_description/meshes/visual/base_link.stl"
-          scale="0.001 0.001 0.001"/>
-</geometry>
-      <material name="gray">
-        <color rgba="0.7 0.7 0.7 1.0"/>
-      </material>
-    </visual>
-  </link>
-  <xacro:rocker
-    name="left_rocker"
-    parent="base_link"
-    xyz="${rocker_x} ${rocker_y} ${rocker_z}"/>
-<xacro:rocker
-    name="right_rocker"
-    parent="base_link"
-    xyz="${rocker_x} ${-rocker_y} ${rocker_z}"/>
-  <xacro:bogie
+    <!-- Includes -->
+    <xacro:include filename="$(find my_rover_description)/urdf/links/base_link.xacro"/>
+    <xacro:include filename="$(find my_rover_description)/urdf/links/rocker.xacro"/>
+    <xacro:include filename="$(find my_rover_description)/urdf/links/bogie.xacro"/>
+    <xacro:include filename="$(find my_rover_description)/urdf/links/wheel.xacro"/>
+    <xacro:include filename="$(find my_rover_description)/urdf/properties.xacro"/>
+    <!-- Base -->
+    <xacro:base_link/>
+    <!-- ================================================= -->
+    <!-- ROCKERS                                             -->
+    <!-- ================================================= -->
+    <xacro:rocker
+        name="left_rocker"
+        parent="base_link"
+        xyz="-0.1037985 0.1413 0.02"
+        rpy="1.5708 0 0"/>
+    <xacro:rocker
+        name="right_rocker"
+        parent="base_link"
+        xyz="-0.1037985 -0.1413 0.02"
+        rpy="1.5708 0 0"/>
+    <!-- ================================================= -->
+    <!-- BOGIES                                              -->
+    <!-- ================================================= -->
+   <xacro:bogie
     name="left_bogie"
     parent="left_rocker"
-    xyz="${bogie_x} ${bogie_y} ${bogie_z}"/>
-<xacro:bogie
+    xyz="0.26214225 -0.20  -0.10"
+    rpy="3.14159 0 0"/>
+   <xacro:bogie
     name="right_bogie"
     parent="right_rocker"
-    xyz="${bogie_x} ${bogie_y} ${bogie_z}"/>
+    xyz="0.26214225 -0.20 -0.08"
+    rpy="-3.14159 0 0"/>
+    <!-- ================================================= -->
+    <!-- rear left                                 -->
+    <!-- ================================================= -->
+    <xacro:wheel
+        name="left_rear_wheel"
+        parent="left_rocker"
+        xyz="-0.25707953 -0.22712987 0"
+        rpy="0 0 0"/>
+    <!-- ================================================= -->
+    <!-- rear right                                   -->
+    <!-- ================================================= -->
+    <xacro:wheel
+        name="right_rear_wheel"
+        parent="right_rocker"
+        xyz="-0.25707953 -0.22712987 0"
+        rpy="0 0 0"/>
+<!-- ================================================= -->
+    <!-- RIGHT REAR                                         -->
+    <!-- ================================================= -->
+    <xacro:wheel
+        name="right_middle_wheel"
+        parent="right_bogie"
+        xyz="-0.195206085 0.025 -0.100411217"
+        rpy="0 0 0"/>
+    <!-- ================================================= -->
+    <!-- LEFT REAR                                          -->
+    <!-- ================================================= -->
+    <xacro:wheel
+        name="left_middle_wheel"
+        parent="left_bogie"
+        xyz="-0.195206085 0.025 -0.100411217"
+        rpy="0 0 0"/>
+    <!-- ================================================= -->
+    <!-- RIGHT MIDDLE                                       -->
+    <!-- ================================================= -->
+    <xacro:wheel
+        name="right_front_wheel"
+        parent="right_bogie"
+        xyz="0.157949245 0.025 -0.130411217"
+        rpy="0 0 0"/>
+    <!-- ================================================= -->
+    <!-- LEFT                                        -->
+    <!-- ================================================= -->
+    <xacro:wheel
+        name="left_front_wheel"
+        parent="left_bogie"
+        xyz="0.157949245 0.025 -0.100411217"
+        rpy="0 0 0"/>
 </robot>

Commit message: Fix Gazebo rover control and simulation launch

File: src/my_rover_description/urdf/my_rover.urdf.xacro (robot description, xacro)
@@ -84,3 +84,96 @@
         xyz="0.157949245 0.025 -0.100411217"
         rpy="0 0 0"/>
+  <!-- Simulated LiDAR -->
+  <link name="lidar_link">
+    <visual>
+      <geometry>
+        <cylinder radius="0.04" length="0.05"/>
+      </geometry>
+    </visual>
+    <collision>
+      <geometry>
+        <cylinder radius="0.04" length="0.05"/>
+      </geometry>
+    </collision>
+    <inertial>
+      <mass value="0.1"/>
+      <inertia
+        ixx="0.0001"
+        ixy="0.0"
+        ixz="0.0"
+        iyy="0.0001"
+        iyz="0.0"
+        izz="0.0001"/>
+    </inertial>
+  </link>
+  <joint name="lidar_joint" type="fixed">
+    <parent link="base_link"/>
+    <child link="lidar_link"/>
+    <origin xyz="0 0 0.30" rpy="0 0 0"/>
+  </joint>
+    <gazebo reference="lidar_link">
+    <sensor name="lidar" type="gpu_lidar">
+  <topic>/scan</topic>
+  <update_rate>10</update_rate>
+  <ray>
+    <scan>
+      <horizontal>
+        <samples>360</samples>
+        <resolution>1</resolution>
+        <min_angle>-3.14159</min_angle>
+        <max_angle>3.14159</max_angle>
+      </horizontal>
+    </scan>
+    <range>
+      <min>0.12</min>
+      <max>12.0</max>
+      <resolution>0.01</resolution>
+    </range>
+  </ray>
+  <always_on>true</always_on>
+  <visualize>true</visualize>
+</sensor>
+  </gazebo>
+  <ros2_control name="GazeboSystem" type="system">
+    <hardware>
+      <plugin>gz_ros2_control/GazeboSimSystem</plugin>
+    </hardware>
+    <joint name="left_front_wheel_joint">
+      <command_interface name="velocity"/>
+      <state_interface name="position"/>
+      <state_interface name="velocity"/>
+    </joint>
+    <joint name="left_middle_wheel_joint">
+      <command_interface name="velocity"/>
+      <state_interface name="position"/>
+      <state_interface name="velocity"/>
+    </joint>
+    <joint name="left_rear_wheel_joint">
+      <command_interface name="velocity"/>
+      <state_interface name="position"/>
+      <state_interface name="velocity"/>
+    </joint>
+    <joint name="right_front_wheel_joint">
+      <command_interface name="velocity"/>
+      <state_interface name="position"/>
+      <state_interface name="velocity"/>
+    </joint>
+    <joint name="right_middle_wheel_joint">
+      <command_interface name="velocity"/>
+      <state_interface name="position"/>
+      <state_interface name="velocity"/>
+    </joint>
+    <joint name="right_rear_wheel_joint">
+      <command_interface name="velocity"/>
+      <state_interface name="position"/>
+      <state_interface name="velocity"/>
+    </joint>
+  </ros2_control>
+    <gazebo>
+    <plugin
+      filename="gz_ros2_control-system"
+      name="gz_ros2_control::GazeboSimROS2ControlPlugin">
+      <parameters>$(find my_rover_description)/config/ros2_controllers.yaml</parameters>
+    </plugin>
+  </gazebo>
 </robot>
